Commit message: Changes to be committed: 	modified:   README.md 	modified:   gluon/urdf/gluon.urdf 	modified:   gluon_control/config/gluon_controllers.yaml 	new file:   gluon_control/config/gluon_spacenav_config.yaml 	new file:   gluon_control/launch/control_by_spacenav.launch 	new file:   gluon_control/launch/gluon_control_position.launch 	renamed:    gluon_control/launch/gluon_control.launch -> gluon_control/launch/gluon_control_trajectory.launch 	new file:   gluon_control/launch/spacenav_gluon.launch 	modified:   gluon_control/src/gluon_hw_interface.cpp 	modified:   gluon_moveit_config/config/joint_limits.yaml

File: gluon/urdf/gluon.urdf (robot description, URDF)
Before this commit: robot gluon, 8 links, 7 joints
Joints:
- joint axis_joint_1: limit lower=-2.79 upper=2.79 effort=30 velocity=3.14 -> lower=-2.79 upper=2.79 effort=30 velocity=6.28
- joint axis_joint_2: limit lower=-1.54 upper=1.54 effort=30 velocity=3.14 -> lower=-1.54 upper=1.54 effort=30 velocity=12.56
- joint axis_joint_3: limit lower=-2.79 upper=2.79 effort=30 velocity=3.14 -> lower=-2.79 upper=2.79 effort=30 velocity=12.56
- joint axis_joint_4: limit lower=-2.79 upper=2.79 effort=30 velocity=3.14 -> lower=-2.79 upper=2.79 effort=30 velocity=12.56
- joint axis_joint_5: limit lower=-2.79 upper=2.79 effort=30 velocity=3.14 -> lower=-2.79 upper=2.79 effort=30 velocity=12.56
- joint axis_joint_6: limit lower=-2.79 upper=2.79 effort=30 velocity=3.14 -> lower=-2.79 upper=2.79 effort=30 velocity=12.56
